File: encoder-tester/encoder-tester.brd (EAGLE design)
At the start: 114.3 x 64.4 mm, 10 parts

Commit message: board fixups
Parts:
- moved J1 12.7 mm to (16.5, 7.62), turned to 90 degrees
- moved J2 7.41 mm to (16.5, 19.1), turned to 90 degrees
Routing:
- net LED2: track 100.1 -> 83.1 mm
- net VIN: track 115.9 -> 128.7 mm
- net LED1: track 86.1 -> 92.4 mm
- net ENC3B: track 69.1 -> 71.3 mm
- net ENC2A: track 44.4 -> 43.0 mm
- net ENC3A: track 71.6 -> 72.4 mm
- net ENC2B: track 40.4 -> 41.2 mm
- added copper zone on layer 16, net GND
- removed copper zone on layer 1, net GND
