File: encoder-tester/encoder-testerB.brd (EAGLE design)
At the start: 121.9 x 64.4 mm, 12 parts, among them J3 POWER_JACKPTH_LOCK

Commit message: update
Parts:
- added C2: (no value), adafruit:E3,5-8
- added J4: (no value), SparkFun-Connectors:1X03
- added R1, R2: 1k, SparkFun-Resistors:AXIAL-0.3
- moved S4 106.7 mm to (110.5, 41.9), turned to 180 degrees
- moved B1 71.2 mm to (86.4, 34.3), turned to 90 degrees
- moved J3 53.9 mm to (125.0, 25.9), turned to 270 degrees
- moved J2 51.7 mm to (22.9, 31.8), turned to 270 degrees
- moved J1 30.7 mm to (22.9, 40.6), turned to 270 degrees
- moved U$3 19.1 mm to (118.1, 41.9)
- moved U$4 19.1 mm to (3.81, 41.9)
- moved S1 6.48 mm to (96.5, 10.2)
- moved S2 6.35 mm to (61.0, 10.2)
- moved S3 6.35 mm to (25.4, 10.2)
Connections:
- new net BUT3: S3.SW-
- new net N$1: J1.2, R1.P$2
- new net N$2: J2.2, R2.P$2
- new net N$3: B1.2, J4.2
- new net N$4: B1.1, J4.3
- net GND: now also C2.-, J4.1, S3.SW+
- net LED1: now also R1.P$1; no longer J1.2
- net LED2: now also R2.P$1; no longer J2.2
- net VIN: now also C2.+
Routing:
- net ENC1B: track 84.2 -> 21.7 mm
- net ENC1A: track 78.1 -> 19.4 mm
- net ENC3A: track 9.54 -> 54.4 mm
- net ENC3B: track 17.5 -> 52.5 mm
- net GND: track 28.5 -> 0.00 mm, vias 2 -> 0
- net LED1: track 32.3 -> 60.3 mm
- net ENC2B: track 49.3 -> 22.0 mm
- net VIN: track 103.9 -> 130.7 mm
- net ENC2A: track 44.4 -> 25.0 mm
- net RESET: track 31.5 -> 19.3 mm
- net N$2: track 0.00 -> 5.08 mm
- net N$1: track 0.00 -> 5.08 mm
- net N$4: track 0.00 -> 5.08 mm
- net N$3: track 0.00 -> 5.08 mm
- net LED2: track 53.9 -> 53.3 mm
Other:
- board size 121.9 x 64.4 mm -> 121.9 x 45.4 mm

Commit message: added second encoder test sketch
Parts:
- added J5: (no value), SparkFun-Connectors:USB-B-MICRO-SMD
- moved J3 1.02 mm to (125.0, 24.9)
Connections:
- net GND: now also J5.GND
- net VIN: now also J5.VBUS
Routing:
- net VIN: track 130.7 -> 137.8 mm
- net GND: track 0.00 -> 4.15 mm
Changed lines of the file:
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@@
 <element name="U$3" library="SparkFun-Hardware" package="STAND-OFF" value="" x="118.11" y="41.91" rot="R180"/>
 <element name="U$4" library="SparkFun-Hardware" package="STAND-OFF" value="" x="3.81" y="41.91" rot="R180"/>
-<element name="J3" library="SparkFun-Connectors" package="POWER_JACK_PTH_LOCK" value="POWER_JACKPTH_LOCK" x="124.968" y="25.908" rot="MR270">
-<attribute name="SF_ID" value="PRT-00119" x="124.968" y="25.908" size="1.778" layer="28" rot="MR270" display="off"/>
-<attribute name="PROD_ID" value="CONN-08197" x="124.968" y="25.908" size="1.778" layer="28" rot="MR270" display="off"/>
+<element name="J3" library="SparkFun-Connectors" package="POWER_JACK_PTH_LOCK" value="POWER_JACKPTH_LOCK" x="124.968" y="24.892" rot="MR270">
+<attribute name="SF_ID" value="PRT-00119" x="124.968" y="24.892" size="1.778" layer="28" rot="MR270" display="off"/>
+<attribute name="PROD_ID" value="CONN-08197" x="124.968" y="24.892" size="1.778" layer="28" rot="MR270" display="off"/>
 </element>
 <element name="S4" library="SparkFun-Switches" package="TACTILE_SWITCH_PTH_6.0MM" value="tact6mm" x="110.49" y="41.91" rot="MR180">
@@
 <element name="J4" library="SparkFun-Connectors" package="1X03" value="" x="93.98" y="31.75" rot="MR180"/>
 <element name="C2" library="adafruit" package="E3,5-8" value="" x="11.43" y="31.75" rot="MR0"/>
+<element name="J5" library="SparkFun-Connectors" package="USB-B-MICRO-SMD" value="" x="119.888" y="34.29" rot="R180">
+<attribute name="PROD_ID" value="CONN-11752" x="119.888" y="34.29" size="1.778" layer="27" rot="R180" display="off"/>
+</element>
 </elements>
 <signals>
@@
 <contactref element="J4" pad="1"/>
 <contactref element="C2" pad="-"/>
+<contactref element="J5" pad="GND"/>
+<wire x1="117.163" y1="35.59" x2="113.06" y2="35.59" width="0.4064" layer="1"/>
+<wire x1="113.06" y1="35.59" x2="113.03" y2="35.56" width="0.254" layer="1"/>
 </signal>
 <signal name="ENC1A">
@@
 <contactref element="S1" pad="B"/>
 <contactref element="B1" pad="7"/>
-<wire x1="83.82" y1="26.67" x2="83.82" y2="23.368" width="1.016" layer="1"/>
-<wire x1="83.82" y1="23.368" x2="87.376" y2="19.812" width="1.016" layer="1"/>
-<wire x1="87.376" y1="19.812" x2="90.424" y2="19.812" width="1.016" layer="1"/>
+<wire x1="83.82" y1="26.67" x2="83.82" y2="22.606" width="1.016" layer="1"/>
+<wire x1="83.82" y1="22.606" x2="86.614" y2="19.812" width="1.016" layer="1"/>
+<wire x1="86.614" y1="19.812" x2="90.424" y2="19.812" width="1.016" layer="1"/>
 <wire x1="90.424" y1="19.812" x2="98.298" y2="19.812" width="1.016" layer="1"/>
 <wire x1="98.298" y1="19.812" x2="99.06" y2="19.05" width="1.016" layer="1"/>
@@
 <contactref element="B1" pad="24"/>
 <contactref element="J3" pad="PWR"/>
-<wire x1="111.0902" y1="25.908" x2="111.0902" y2="33.6898" width="2.54" layer="1"/>
+<wire x1="111.0902" y1="24.892" x2="111.0902" y2="33.02" width="2.54" layer="1"/>
+<wire x1="111.0902" y1="33.02" x2="111.0902" y2="33.6898" width="2.54" layer="1"/>
 <wire x1="111.0902" y1="33.6898" x2="109.22" y2="35.56" width="2.54" layer="1"/>
 <wire x1="109.22" y1="35.56" x2="104.14" y2="35.56" width="2.54" layer="1"/>
@@
 <wire x1="19.05" y1="40.64" x2="19.05" y2="41.91" width="2.54" layer="1"/>
 <wire x1="22.86" y1="40.64" x2="22.86" y2="41.91" width="2.54" layer="1"/>
+<contactref element="J5" pad="VBUS"/>
+<wire x1="117.163" y1="32.99" x2="111.1202" y2="32.99" width="0.4064" layer="1"/>
+<wire x1="111.1202" y1="32.99" x2="111.0902" y2="33.02" width="0.254" layer="1"/>
 </signal>
 <signal name="LED1">
